Commit message: robot model works in env

File: models/robots/model.urdf (robot description, URDF)
Before this commit: robot panda, 12 links, 11 joints
Links:
- link panda_hand: geometry collision mesh filename=../meshes/collision/hand.stl; visual mesh filename=../meshes/visual/hand.dae
- link panda_leftfinger: geometry collision mesh filename=../meshes/collision/finger.stl; visual mesh filename=../meshes/visual/finger.dae
- link panda_link0: geometry collision mesh filename=../meshes/collision/link0.stl; visual mesh filename=../meshes/visual/link0.dae
- link panda_link1: geometry collision mesh filename=../meshes/collision/link1.stl; visual mesh filename=../meshes/visual/link1.dae
- link panda_link2: geometry collision mesh filename=../meshes/collision/link2.stl; visual mesh filename=../meshes/visual/link2.dae
- link panda_link3: geometry collision mesh filename=../meshes/collision/link3.stl; visual mesh filename=../meshes/visual/link3.dae
- link panda_link4: geometry collision mesh filename=../meshes/collision/link4.stl; visual mesh filename=../meshes/visual/link4.dae
- link panda_link5: geometry collision mesh filename=../meshes/collision/link5.stl; visual mesh filename=../meshes/visual/link5.dae
- link panda_link6: geometry collision mesh filename=../meshes/collision/link6.stl; visual mesh filename=../meshes/visual/link6.dae
- link panda_link7: geometry collision mesh filename=../meshes/collision/link7.stl; visual mesh filename=../meshes/visual/link7.dae
- link panda_rightfinger: geometry collision mesh filename=../meshes/collision/finger.stl; visual mesh filename=../meshes/visual/finger.dae

Commit message: GP classification of bad model points kinda works

File: models/robots/model.urdf (robot description, URDF)
Before this commit: robot panda, 12 links, 11 joints
Links:
- removed link panda_link0
- added link base_link; collision mesh filename=../meshes/collision/link0.stl; visual mesh filename=../meshes/visual/link0.dae
Joints:
- joint panda_joint1: parent panda_link0 -> base_link
